File: pcb/motordriver/motordriver.kicad_sch (KiCad schematic)
At the start: 15 parts, among them J1 Conn_01x03_Pin, J2 Conn_01x02_Pin, J3 Conn_01x02_Pin, J4 Conn_01x03_Pin, U1 ESP32-CAM, U2 DRV8833PWP

Commit message: PCB created
Parts:
- removed J1, J4: Conn_01x03_Pin, Connector_PinHeader_2.54mm:PinHeader_1x03_P2.54mm_Horizontal, symbol Connector:Conn_01x03_Pin
- removed J2, J3: Conn_01x02_Pin, Connector_PinHeader_2.54mm:PinHeader_1x02_P2.54mm_Vertical, symbol Connector:Conn_01x02_Pin
- removed U1: ESP32-CAM, _for_motordriver:ESP32-CAM, symbol _for_motordriver:ESP32-CAM_Alt1
- added C5, C6: 22uF, Capacitor_SMD:C_1206_3216Metric, symbol Device:C
- added H1, H2, H3: (no value), PCM_JLCPCB:Hole_Tooling_JLCPCB, symbol PCM_JLCPCB-Manufacturing:Tooling Hole, PCM_JLCPCB, 1.152mm
- added J1: USB_C_Receptacle_PowerOnly_6P, Connector_USB:USB_C_Receptacle_HRO_TYPE-C-31-M-17, symbol Connector:USB_C_Receptacle_PowerOnly_6P
- added J2, J3: Conn_01x08_Pin, Connector_PinSocket_2.54mm:PinSocket_1x08_P2.54mm_Vertical, symbol Connector:Conn_01x08_Pin
- added J4, J5: Conn_02x03_Odd_Even, Connector_PinHeader_2.54mm:PinHeader_2x03_P2.54mm_Horizontal, symbol Connector_Generic:Conn_02x03_Odd_Even
- added R6, R7: 5k1, Resistor_SMD:R_0603_1608Metric, symbol Device:R
- C1: LCSC (none) -> C377773
- C2: renamed from C3; LCSC (none) -> C57112
- C3: renamed from C2; value 10uF -> 22uF; footprint Capacitor_SMD:C_1210_3225Metric -> Capacitor_SMD:C_1206_3216Metric; LCSC (none) -> C12891
- C4: value 10uF -> 22uF; footprint Capacitor_SMD:C_1210_3225Metric -> Capacitor_SMD:C_1206_3216Metric; LCSC (none) -> C12891
- R1, R2, R3, R4, R5: LCSC (none) -> C327006
- U2: LCSC (none) -> C50506
Connections:
- net +5V: now also R5.2, J1.A9 (VBUS), J1.B9 (VBUS), J2.1 (Pin_1); no longer R5.1
- net GND: now also C5.2, C6.2, J1.A12 (GND), J1.B12 (GND), J2.2 (Pin_2), J3.1 (Pin_1), J3.5 (Pin_5), J4.6 (Pin_6), J5.6 (Pin_6), R6.2, R7.2
- net MotorL1: now also J2.5 (Pin_5)
- net MotorL2: now also J2.6 (Pin_6)
- net MotorR1: now also J2.3 (Pin_3)
- net MotorR2: now also J2.4 (Pin_4)
- net Servo1: now also J2.7 (Pin_7), J5.2 (Pin_2)
- net Servo2: now also J3.3 (Pin_3), J4.2 (Pin_2)
- net at U2.5 (BOUT2): now also J5.5 (Pin_5)
- net at U2.7 (BOUT1): now also J5.3 (Pin_3)
- net at U2.4 (AOUT2): now also J4.5 (Pin_5)
- net at U2.2 (AOUT1): now also J4.3 (Pin_3)
- net at R4.2: now also C6.1, J5.4 (Pin_4)
- new net: J1.A5 (CC1), R7.1
- new net: C5.1, J4.4 (Pin_4), R5.1
- new net: J1.B5 (CC2), R6.1
Other:
- note added: "Manually cut away Pin 1 of J4 and J5"
- note removed: "ESP-CAM kann natürlich gegen 2 Pinheaderbuchsen getauscht werden."
- note removed: "USB C Buchse hier"
- company: (none) -> Hackerspace-FFM e.V.
- title: (none) -> Motor driver for ESP-CAM
- moved on the sheet: C1, C2, C3, C4, R1, R2, R3, R4, R5, U2

Commit message: Updated PCB, fixed minor bugs on PCB
Parts:
- added PN1: (no value), PCM_JLCPCB:Part_Num_JLCPCB, symbol PCM_JLCPCB-Manufacturing:Part Number, PCM_JLCPCB, 0.8x0.15mm
Connections:
- net GND: no longer J3.1 (Pin_1)
Other:
- note added: "On some boards pin 9 is not GND but GND/R. GND here then keeps board in Reset."
Changed lines of the file:
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@@
 	(title_block
 		(title "Motor driver for ESP-CAM")
-		(date "2026-05-16")
-		(rev "1")
+		(date "2026-05-26")
+		(rev "2")
 		(company "Hackerspace-FFM e.V.")
 		(comment 1 "2026-05 by Lutz Lisseck")
@@
 		)
 	)
+	(text "On some boards pin 9 is not\nGND but GND/R. GND here then\nkeeps board in Reset."
+		(exclude_from_sim no)
+		(at 116.332 55.372 0)
+		(effects
+			(font
+				(size 1.27 1.27)
+			)
+		)
+	)
 	(junction
 		(at 43.18 19.05)
@@
 	)
 	(junction
-		(at 121.92 43.18)
-		(diameter 0)
-		(color 0 0 0 0)
-	)
-	(junction
 		(at 46.99 19.05)
 		(diameter 0)
@@
 	(wire
 		(pts
-			(xy 121.92 33.02) (xy 121.92 43.18)
-		)
-		(stroke
-			(width 0)
-			(type default)
-		)
-	)
-	(wire
-		(pts
 			(xy 72.39 76.2) (xy 78.74 76.2)
 		)
@@
 	(wire
 		(pts
-			(xy 121.92 43.18) (xy 121.92 44.45)
+			(xy 121.92 33.02) (xy 121.92 44.45)
 		)
 		(stroke
@@
 		(pts
 			(xy 152.4 88.9) (xy 152.4 92.71)
-		)
-		(stroke
-			(width 0)
-			(type default)
-		)
-	)
-	(wire
-		(pts
-			(xy 124.46 43.18) (xy 121.92 43.18)
 		)
 		(stroke
@@
 					(unit 1)
 				)
+			)
+		)
+	)
+	(symbol
+		(lib_id "PCM_JLCPCB-Manufacturing:Part Number, PCM_JLCPCB, 0.8x0.15mm")
+		(at 24.13 132.08 0)
+		(unit 1)
+		(body_style 1)
+		(exclude_from_sim no)
+		(in_bom yes)
+		(on_board yes)
+		(in_pos_files yes)
+		(dnp no)
+		(fields_autoplaced yes)
+		(property "Reference" "PN1"
+			(at 25.4 132.0799 0)
+			(show_name no)
+			(do_not_autoplace no)
+			(effects
+				(font
+					(size 1.27 1.27)
+				)
+				(justify left)
+			)
+		)
+		(property "Value" ""
+			(at 24.13 132.08 0)
+			(show_name no)
+			(do_not_autoplace no)
+			(effects
+				(font
+					(size 1.27 1.27)
+				)
+			)
+		)
+		(property "Footprint" "PCM_JLCPCB:Part_Num_JLCPCB"
+			(at 24.13 132.08 0)
+			(hide yes)
+			(show_name no)
+			(do_not_autoplace no)
+			(effects
+				(font
+					(size 1.27 1.27)
+				)
+			)
+		)
+		(property "Datasheet" "https://jlcpcb.com/help/article/How-to-remove-order-number-from-your-PCB"
+			(at 24.13 132.08 0)
+			(hide yes)
+			(show_name no)
+			(do_not_autoplace no)
+			(effects
+				(font
+					(size 1.27 1.27)
+				)
+			)
+		)
+		(property "Description" "To indicate the location, simply add the text \"JLCJLCJLCJLC\" to the silk layer and select the \"Specify a location\" option when placing your order. Please note that if this option is not chosen, we may not notice that you have added the text.   Note: Use only \"JLCJLCJLCJLC\" without any additional characters. The font size should be larger than 0.8mm in height and 0.15mm in width."
+			(at 24.13 132.08 0)
+			(hide yes)
+			(show_name no)
+			(do_not_autoplace no)
+			(effects
+				(font
+					(size 1.27 1.27)
+				)
+			)
+		)
+		(instances
+			(project "motordriver"
+				(path "/feb821bf-a6f8-4c58-978a-b64215145b9d"
+					(reference "PN1")
+					(unit 1)
+				)
